File: Design Files/ADA4610 Transimpedance Amplifier/V1.1/ADA4610 Transimpedance Amplifier.kicad_sch (KiCad schematic)
At the start: 33 parts, among them J1 Conn_01x03_Male, J2 Conn_Coaxial, U1 ADA4610-1xR, U2 ADA4610-1xR

Commit message: commit as built 2022-12-27
As built, working with +5V unipolar and ~100x second stage gain. IRDA signals clearly visible at 37KHz.
Parts:
- added C?: 10nF, symbol Device:C
- added R? (x2): 10k, Resistor_SMD:R_0603_1608Metric_Pad0.98x0.95mm_HandSolder, symbol Device:R_US
- C2: value 15pF -> 33pF
- C5: value 10u -> 1uF
- C?: value 1nF -> 10nF
- R3, R4: value 10k -> 1k
- R8: value 49.9k -> 100k
Connections:
- net VEE is gone; now on net GND: C2.1, C3.2, C7.2, J1.2 (Pin_2), R1.2, R4.2, TP3.1, U1.2 (V-), U2.2 (V-)
- net GND: now also C?.1, R?.2; no longer R7.1
- net VCC: now also R?.1
- net at C4.2, R6.2, TP5.1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: now also R7.1; no longer U2.3 (+)
- new net: C?.2, R?.1, R?.2, U2.3 (+)
Other:
- note added: "TEMP SHORT FOR UNIPOLAR"
